Commit message: added vanderlande rail to irb6700

File: abb_irb6700_support/urdf/irb6700_200_260_macro.xacro (robot description, xacro)
@@ -4,4 +4,13 @@
     <xacro:include filename="$(find abb_resources)/urdf/common_materials.xacro"/>
     <!-- link list -->
+    <link name="${prefix}actuator_link">
+      <collision>
+        <origin xyz="0 0 0" rpy="0 0 0" />
+        <geometry>
+          <box size="1 8 0.2"/>
+        </geometry>
+        <xacro:material_abb_yellow/>
+      </collision>
+    </link>
     <link name="${prefix}base_link">
       <visual>
@@ -148,6 +157,13 @@
       </collision>
     </link>
+    <joint name="${prefix}actuator_joint" type="prismatic">
+      <origin xyz="0 0 0" rpy="0 0 0" />
+      <parent link="${prefix}actuator_link" />
+      <child link="${prefix}base_link" />
+      <axis xyz="0 1 0" />
+      <limit lower="-4" upper="4" effort="0" velocity="1" />
+    </joint>
     <joint name="${prefix}joint_1" type="revolute">
-      <origin xyz="0 0 0.78" rpy="0 0 0" />
+      <origin xyz="0 0 0.88" rpy="0 0 0" />
       <parent link="${prefix}base_link" />
       <child link="${prefix}link_1" />

Commit message: non-working commit, added transmission and gazebo links to files

File: abb_irb6700_support/urdf/irb6700_200_260_macro.xacro (robot description, xacro)
@@ -3,4 +3,15 @@
   <xacro:macro name="abb_irb6700_200_260" params="prefix">
     <xacro:include filename="$(find abb_resources)/urdf/common_materials.xacro"/>
+    <xacro:include filename="$(find abb_irb6700_support)/urdf/irb6700_200_260.transmission.xacro"/>
+    <xacro:include filename="$(find abb_irb6700_support)/urdf/irb6700_200_260.gazebo.xacro"/>
+    <xacro:macro name="cylinder_inertial" params="radius length mass *origin">
+      <inertial>
+        <mass value="${mass}" />
+        <xacro:insert_block name="origin" />
+        <inertia ixx="${0.0833333 * mass * (3 * radius * radius + length * length)}" ixy="0.0" ixz="0.0"
+        iyy="${0.0833333 * mass * (3 * radius * radius + length * length)}" iyz="0.0"
+        izz="${0.5 * mass * radius * radius}" />
+      </inertial>
+    </xacro:macro>
     <!-- link list -->
     <link name="${prefix}actuator_link">
@@ -12,4 +23,7 @@
         <xacro:material_abb_yellow/>
       </collision>
+      <xacro:cylinder_inertial radius="0.06" length="0.05" mass="10">
+          <origin xyz="0.0 0.0 0.0" rpy="0 0 0" />
+      </xacro:cylinder_inertial>
     </link>
     <link name="${prefix}base_link">
@@ -28,4 +42,7 @@
         <xacro:material_abb_yellow/>
       </collision>
+      <xacro:cylinder_inertial radius="0.06" length="0.05" mass="10">
+          <origin xyz="0.0 0.0 0.0" rpy="0 0 0" />
+      </xacro:cylinder_inertial>
     </link>
     <link name="${prefix}link_1">
@@ -41,36 +58,4 @@
         <geometry>
           <mesh filename="package://abb_irb6700_support/meshes/irb6700/collision/link_1.stl" />
-        </geometry>
-        <xacro:material_abb_yellow/>
-      </collision>
-    </link>
-    <link name="${prefix}cylinder">
-      <visual>
-        <origin xyz="0 0 0" rpy="0 0 0" />
-        <geometry>
-          <mesh filename="package://abb_irb6700_support/meshes/irb6700/visual/cylinder.stl" />
-        </geometry>
-        <xacro:material_abb_white/>
-      </visual>
-      <collision>
-        <origin xyz="0 0 0" rpy="0 0 0" />
-        <geometry>
-          <mesh filename="package://abb_irb6700_support/meshes/irb6700/collision/cylinder.stl" />
-        </geometry>
-        <xacro:material_abb_yellow/>
-      </collision>
-    </link>
-    <link name="${prefix}piston">
-      <visual>
-        <origin xyz="0 0 0" rpy="0 0 0" />
-        <geometry>
-          <mesh filename="package://abb_irb6700_support/meshes/irb6700/visual/piston.stl" />
-        </geometry>
-        <xacro:material_abb_white/>
-      </visual>
-      <collision>
-        <origin xyz="0 0 0" rpy="0 0 0" />
-        <geometry>
-          <mesh filename="package://abb_irb6700_support/meshes/irb6700/collision/piston.stl" />
         </geometry>
         <xacro:material_abb_yellow/>
@@ -206,20 +191,4 @@
       <limit lower="-${radians(360)}" upper="${radians(360)}" effort="0" velocity="${radians(210)}" />
     </joint>
-    <joint name="${prefix}cylinder_joint" type="revolute">
-      <origin xyz="-0.349 -0.194 -0.142" rpy="0 0 0" />
-      <parent link="${prefix}link_1" />
-      <child link="${prefix}cylinder" />
-      <axis xyz="0 1 0" />
-      <mimic joint="${prefix}joint_2" multiplier="-0.25"/>
-      <limit lower="-${radians(65*0.25)}" upper="${radians(85*0.25)}" effort="0" velocity="100" />
-    </joint>
-    <joint name="${prefix}piston_joint" type="prismatic">
-      <origin xyz="0 0 0" rpy="0.20897 0 -${radians(90)}" />
-      <parent link="${prefix}cylinder" />
-      <child link="${prefix}piston" />
-      <axis xyz="0 1 0" />
-      <mimic joint="${prefix}joint_2" multiplier="0.15"/>
-      <limit lower="-0.25" upper="0.25" effort="0" velocity="100" />
-    </joint>
     <!-- ROS-Industrial 'base' frame: base_link to ABB World Coordinates transform -->
     <link name="${prefix}base" />
@@ -243,4 +212,6 @@
       <child link="${prefix}tool0" />
     </joint>
+    <xacro:irb6700_200_260_transmission prefix="${prefix}" />
+    <xacro:irb6700_200_260_gazebo prefix="${prefix}" />
   </xacro:macro>
 </robot>
