Commit message: fixing transmission and inertia values

File: abb_irb6700_support/urdf/irb6700_200_260.transmission.xacro (robot description, xacro)
@@ -5,8 +5,8 @@
         <type>transmission_interface/SimpleTransmission</type>
         <joint name="${prefix}actuator_joint">
-            <hardwareInterface>hardware_interface/EffortJointInterface</hardwareInterface>
+            <hardwareInterface>hardware_interface/PositionJointInterface</hardwareInterface>
         </joint>
         <actuator name="actuator_joint_motor">
-            <hardwareInterface>hardware_interface/EffortJointInterface</hardwareInterface>
+            <hardwareInterface>hardware_interface/PositionJointInterface</hardwareInterface>
             <mechanicalReduction>1</mechanicalReduction>
         </actuator>
@@ -15,8 +15,8 @@
         <type>transmission_interface/SimpleTransmission</type>
         <joint name="${prefix}joint_1">
-            <hardwareInterface>hardware_interface/EffortJointInterface</hardwareInterface>
+            <hardwareInterface>hardware_interface/PositionJointInterface</hardwareInterface>
         </joint>
         <actuator name="joint_1_motor">
-            <hardwareInterface>hardware_interface/EffortJointInterface</hardwareInterface>
+            <hardwareInterface>hardware_interface/PositionJointInterface</hardwareInterface>
             <mechanicalReduction>1</mechanicalReduction>
         </actuator>
@@ -25,8 +25,8 @@
         <type>transmission_interface/SimpleTransmission</type>
         <joint name="${prefix}joint_2">
-            <hardwareInterface>hardware_interface/EffortJointInterface</hardwareInterface>
+            <hardwareInterface>hardware_interface/PositionJointInterface</hardwareInterface>
         </joint>
         <actuator name="joint_2_motor">
-            <hardwareInterface>hardware_interface/EffortJointInterface</hardwareInterface>
+            <hardwareInterface>hardware_interface/PositionJointInterface</hardwareInterface>
             <mechanicalReduction>1</mechanicalReduction>
         </actuator>
@@ -35,8 +35,8 @@
         <type>transmission_interface/SimpleTransmission</type>
         <joint name="${prefix}joint_3">
-            <hardwareInterface>hardware_interface/EffortJointInterface</hardwareInterface>
+            <hardwareInterface>hardware_interface/PositionJointInterface</hardwareInterface>
         </joint>
         <actuator name="joint_3_motor">
-            <hardwareInterface>hardware_interface/EffortJointInterface</hardwareInterface>
+            <hardwareInterface>hardware_interface/PositionJointInterface</hardwareInterface>
             <mechanicalReduction>1</mechanicalReduction>
         </actuator>
@@ -45,8 +45,8 @@
         <type>transmission_interface/SimpleTransmission</type>
         <joint name="${prefix}joint_4">
-            <hardwareInterface>hardware_interface/EffortJointInterface</hardwareInterface>
+            <hardwareInterface>hardware_interface/PositionJointInterface</hardwareInterface>
         </joint>
         <actuator name="joint_4_motor">
-            <hardwareInterface>hardware_interface/EffortJointInterface</hardwareInterface>
+            <hardwareInterface>hardware_interface/PositionJointInterface</hardwareInterface>
             <mechanicalReduction>1</mechanicalReduction>
         </actuator>
@@ -55,8 +55,8 @@
         <type>transmission_interface/SimpleTransmission</type>
         <joint name="${prefix}joint_5">
-            <hardwareInterface>hardware_interface/EffortJointInterface</hardwareInterface>
+            <hardwareInterface>hardware_interface/PositionJointInterface</hardwareInterface>
         </joint>
         <actuator name="joint_5_motor">
-            <hardwareInterface>hardware_interface/EffortJointInterface</hardwareInterface>
+            <hardwareInterface>hardware_interface/PositionJointInterface</hardwareInterface>
             <mechanicalReduction>1</mechanicalReduction>
         </actuator>
@@ -65,8 +65,8 @@
         <type>transmission_interface/SimpleTransmission</type>
         <joint name="${prefix}joint_6">
-            <hardwareInterface>hardware_interface/EffortJointInterface</hardwareInterface>
+            <hardwareInterface>hardware_interface/PositionJointInterface</hardwareInterface>
         </joint>
         <actuator name="joint_6_motor">
-            <hardwareInterface>hardware_interface/EffortJointInterface</hardwareInterface>
+            <hardwareInterface>hardware_interface/PositionJointInterface</hardwareInterface>
             <mechanicalReduction>1</mechanicalReduction>
         </actuator>

File: abb_irb6700_support/urdf/irb6700_200_260_macro.xacro (robot description, xacro)
@@ -61,4 +61,7 @@
         <xacro:material_abb_yellow/>
       </collision>
+      <xacro:cylinder_inertial radius="0.06" length="0.05" mass="10">
+          <origin xyz="0.0 0.0 0.0" rpy="0 0 0" />
+      </xacro:cylinder_inertial>
     </link>
     <link name="${prefix}link_2">
@@ -77,4 +80,7 @@
         <xacro:material_abb_yellow/>
       </collision>
+      <xacro:cylinder_inertial radius="0.06" length="0.05" mass="10">
+          <origin xyz="0.0 0.0 0.0" rpy="0 0 0" />
+      </xacro:cylinder_inertial>
     </link>
     <link name="${prefix}link_3">
@@ -93,4 +99,7 @@
         <xacro:material_abb_yellow/>
       </collision>
+      <xacro:cylinder_inertial radius="0.06" length="0.05" mass="10">
+          <origin xyz="0.0 0.0 0.0" rpy="0 0 0" />
+      </xacro:cylinder_inertial>
     </link>
     <link name="${prefix}link_4">
@@ -109,4 +118,7 @@
         <xacro:material_abb_yellow/>
       </collision>
+      <xacro:cylinder_inertial radius="0.06" length="0.05" mass="5">
+          <origin xyz="0.0 0.0 0.0" rpy="0 0 0" />
+      </xacro:cylinder_inertial>
     </link>
     <link name="${prefix}link_5">
@@ -125,4 +137,7 @@
         <xacro:material_abb_yellow/>
       </collision>
+      <xacro:cylinder_inertial radius="0.06" length="0.05" mass="2">
+          <origin xyz="0.0 0.0 0.0" rpy="0 0 0" />
+      </xacro:cylinder_inertial>
     </link>
     <link name="${prefix}link_6">
@@ -141,4 +156,7 @@
         <xacro:material_abb_yellow/>
       </collision>
+      <xacro:cylinder_inertial radius="0.06" length="0.05" mass="1">
+          <origin xyz="0.0 0.0 0.0" rpy="0 0 0" />
+      </xacro:cylinder_inertial>
     </link>
     <joint name="${prefix}actuator_joint" type="prismatic">
@@ -213,5 +231,5 @@
     </joint>
     <xacro:irb6700_200_260_transmission prefix="${prefix}" />
-    <xacro:irb6700_200_260_gazebo prefix="${prefix}" />
+<!--    <xacro:irb6700_200_260_gazebo prefix="${prefix}" />-->
   </xacro:macro>
 </robot>
